Commit message: chanded collision masks

File: franka_description/robots/panda_arm.xacro (robot description, xacro)
@@ -43,11 +43,11 @@
       </visual>
       <collision>
-        <origin xyz="0 0 -0.1915" rpy="0 0 0"/>
-        <geometry>
-          <cylinder radius="${0.06+safety_distance}" length="0.2830" />
-        </geometry>
-      </collision>
-      <collision>
-        <origin xyz="0 0 -0.333" rpy="0 0 0"/>
+        <origin xyz="0 0 -0.1465" rpy="0 0 0"/>
+        <geometry>
+          <cylinder radius="${0.06+safety_distance}" length="0.1930" />
+        </geometry>
+      </collision>
+      <collision>
+        <origin xyz="0 0 -0.243" rpy="0 0 0"/>
         <geometry>
           <sphere radius="${0.06+safety_distance}" />
@@ -286,22 +286,4 @@
     </joint>
     <link name="${arm_id}_link8">
-      <collision>
-        <origin xyz="0.0424 0.0424 -0.0250" rpy="${pi} ${pi/2} ${pi/2}"/>
-        <geometry>
-          <cylinder radius="${0.03+safety_distance}"  length="0.01" />
-        </geometry>
-      </collision>
-      <collision>
-        <origin xyz="0.0424 0.0424 -0.02" rpy="0 0 0"/>
-        <geometry>
-          <sphere radius="${0.03+safety_distance}"  />
-        </geometry>
-      </collision>
-      <collision>
-        <origin xyz="0.0424 0.0424 -0.03" rpy="0 0 0"/>
-        <geometry>
-          <sphere radius="${0.03+safety_distance}"  />
-        </geometry>
-      </collision>
     </link>
     <joint name="${arm_id}_joint8" type="fixed">
